Commit message: Fix inertial/mass values to approximately correct.

File: urdf/ar_gripper_macro.xacro (robot description, xacro)
@@ -21,4 +21,8 @@
         <origin rpy="0.0 0.0 0.0" xyz="0 0 0"/>
       </collision>
+      <inertial>
+        <mass value="0.040" />
+        <inertia ixx="1.0" ixy="0.0" ixz="0.0" iyy="1.0" iyz="0.0" izz="1.0"/>
+      </inertial>
     </link>
     <link name="${prefix}ar_gripper_body">
@@ -37,4 +41,8 @@
         <origin rpy="0.0 0.0 0.0" xyz="0 0 0"/>
       </collision>
+      <inertial>
+        <mass value="0.400" />
+        <inertia ixx="1.0" ixy="0.0" ixz="0.0" iyy="1.0" iyz="0.0" izz="1.0"/>
+      </inertial>
     </link>
     <link name="${prefix}ar_gripper_finger1">
@@ -54,5 +62,5 @@
       </collision>
       <inertial>
-        <mass value="100"/>
+        <mass value="0.040"/>
         <inertia ixx="1.0" ixy="0.0" ixz="0.0" iyy="1.0" iyz="0.0" izz="1.0"/>
       </inertial>
@@ -74,5 +82,5 @@
       </collision>
       <inertial>
-        <mass value="100"/>
+        <mass value="0.040"/>
         <inertia ixx="1.0" ixy="0.0" ixz="0.0" iyy="1.0" iyz="0.0" izz="1.0"/>
       </inertial>

Commit message: Change commands from percent to actual values. Change finger direction so 0 is closed and 0.05 is opened. Deprecate sim node in favor of ros_control in Gazebo (not yet finished). Untested on real hardware.

File: urdf/ar_gripper_macro.xacro (robot description, xacro)
@@ -1,4 +1,5 @@
 <?xml version="1.0" encoding="UTF-8"?>
-<robot name="ar_gripper" xmlns:xacro="http://ros.org/wiki/xacro">
+<robot name="ar_gripper"
+  xmlns:xacro="http://ros.org/wiki/xacro">
   <xacro:macro name="ar_gripper_macro" params="prefix">
     <material name="${prefix}Black">
@@ -23,5 +24,6 @@
       <inertial>
         <mass value="0.040" />
-        <inertia ixx="1.0" ixy="0.0" ixz="0.0" iyy="1.0" iyz="0.0" izz="1.0"/>
+        <!-- These numbers are not correct -->
+        <inertia ixx="0.001" ixy="0.0" ixz="0.0" iyy="0.001" iyz="0.0" izz="0.001"/>
       </inertial>
     </link>
@@ -43,5 +45,6 @@
       <inertial>
         <mass value="0.400" />
-        <inertia ixx="1.0" ixy="0.0" ixz="0.0" iyy="1.0" iyz="0.0" izz="1.0"/>
+        <!-- These numbers are not correct -->
+        <inertia ixx="0.001" ixy="0.0" ixz="0.0" iyy="0.001" iyz="0.0" izz="0.001"/>
       </inertial>
     </link>
@@ -51,5 +54,5 @@
           <mesh filename="package://ar_gripper/meshes/finger.stl"/>
         </geometry>
-        <origin rpy="0.0 0.0 0.0" xyz="0.0 0.0 0.0"/>
+        <origin rpy="0 0 0" xyz="0 0 0"/>
         <material name="${prefix}Black">
         </material>
@@ -59,9 +62,10 @@
           <mesh filename="package://ar_gripper/meshes/finger.stl"/>
         </geometry>
-        <origin rpy="0.0 0.0 0.0" xyz="0.0 0.0 0.0"/>
+        <origin rpy="0 0 0" xyz="0 0 0"/>
       </collision>
       <inertial>
         <mass value="0.040"/>
-        <inertia ixx="1.0" ixy="0.0" ixz="0.0" iyy="1.0" iyz="0.0" izz="1.0"/>
+        <!-- These numbers are not correct -->
+        <inertia ixx="0.001" ixy="0.0" ixz="0.0" iyy="0.001" iyz="0.0" izz="0.001"/>
       </inertial>
     </link>
@@ -71,5 +75,5 @@
           <mesh filename="package://ar_gripper/meshes/finger.stl"/>
         </geometry>
-        <origin rpy="0.0 0.0 0.0" xyz="0.0 0.0 0.0"/>
+        <origin rpy="0 0 0" xyz="0 0 0"/>
         <material name="${prefix}Black">
         </material>
@@ -79,9 +83,10 @@
           <mesh filename="package://ar_gripper/meshes/finger.stl"/>
         </geometry>
-        <origin rpy="0.0 0.0 0.0" xyz="0.0 0.0 0.0"/>
+        <origin rpy="0 0 0" xyz="0 0 0"/>
       </collision>
       <inertial>
         <mass value="0.040"/>
-        <inertia ixx="1.0" ixy="0.0" ixz="0.0" iyy="1.0" iyz="0.0" izz="1.0"/>
+        <!-- These numbers are not correct -->
+        <inertia ixx="0.001" ixy="0.0" ixz="0.0" iyy="0.001" iyz="0.0" izz="0.001"/>
       </inertial>
     </link>
@@ -91,20 +96,20 @@
       <child link="${prefix}ar_gripper_body"/>
       <axis xyz="0 0 0"/>
-      <origin rpy="0.0 0.0 0.0" xyz="0 0 0.006"/>
+      <origin rpy="0 0 0" xyz="0 0 0.006"/>
     </joint>
     <joint name="${prefix}ar_gripper_body_finger1" type="prismatic">
-      <limit effort="1000.0" lower="-0.05" upper="0.0" velocity="1.0"/>
+      <limit effort="1000.0" lower="0.0" upper="0.05" velocity="0.02"/>
       <parent link="${prefix}ar_gripper_body"/>
       <child link="${prefix}ar_gripper_finger1"/>
-      <axis xyz="1 0 0"/>
-      <origin rpy="0.0 0.0 0.0" xyz="0.0 0 0.0756"/>
+      <axis xyz="-1 0 0"/>
+      <origin rpy="0 0 0" xyz="0.0 0 0.0756"/>
     </joint>
     <joint name="${prefix}ar_gripper_body_finger2" type="prismatic">
-      <limit effort="1000.0" lower="-0.05" upper="0.0" velocity="1.0"/>
+      <limit effort="1000.0" lower="0.0" upper="0.05" velocity="0.02"/>
       <parent link="${prefix}ar_gripper_body"/>
       <child link="${prefix}ar_gripper_finger2"/>
-      <axis xyz="1 0 0"/>
+      <axis xyz="-1 0 0"/>
       <mimic joint="${prefix}ar_gripper_body_finger1" multiplier="1.0" offset="0.0" />
-      <origin rpy="0.0 0.0 ${pi}" xyz="0.0 0 0.0756"/>
+      <origin rpy="0 0 ${pi}" xyz="0.0 0 0.0756"/>
     </joint>
   </xacro:macro>

Commit message: Some tweaks and fixes

File: urdf/ar_gripper_macro.xacro (robot description, xacro)
@@ -94,5 +94,5 @@
     </joint>
     <joint name="${prefix}ar_gripper_body_finger1" type="prismatic">
-      <limit effort="1000.0" lower="-0.05" upper="0.0" velocity="1.0"/>
+      <limit effort="1000.0" lower="-0.05" upper="0.0" velocity="0.0031"/>
       <parent link="${prefix}ar_gripper_body"/>
       <child link="${prefix}ar_gripper_finger1"/>
@@ -101,5 +101,5 @@
     </joint>
     <joint name="${prefix}ar_gripper_body_finger2" type="prismatic">
-      <limit effort="1000.0" lower="-0.05" upper="0.0" velocity="1.0"/>
+      <limit effort="1000.0" lower="-0.05" upper="0.0" velocity="0.0031"/>
       <parent link="${prefix}ar_gripper_body"/>
       <child link="${prefix}ar_gripper_finger2"/>
