Commit message: Standardize with `tf_prefix`. Add URDF macro for ros2_control.

File: ar_gripper/srdf/ar_gripper_macro.srdf.xacro (robot description, xacro)
@@ -5,13 +5,13 @@
 -->
 <robot xmlns:xacro="http://wiki.ros.org/xacro">
-  <xacro:macro name="ar_gripper_srdf" params="name prefix">
+  <xacro:macro name="ar_gripper_srdf" params="name tf_prefix">
     <!--GROUPS - Representation of a set of joints and links. This can be useful for specifying DOF to plan for, defining arms, end effectors, etc-->
-    <group name="${prefix}${name}ar_gripper">
-      <link name="${prefix}${name}ar_gripper_adapter" />
-      <link name="${prefix}${name}ar_gripper_body" />
-      <link name="${prefix}${name}ar_gripper_finger1" />
-      <link name="${prefix}${name}ar_gripper_finger2" />
-      <joint name="${prefix}${name}ar_gripper_body_finger1" />
-      <passive_joint name="${prefix}${name}ar_gripper_body_finger2" />
+    <group name="${tf_prefix}${name}ar_gripper">
+      <link name="${tf_prefix}${name}ar_gripper_adapter" />
+      <link name="${tf_prefix}${name}ar_gripper_body" />
+      <link name="${tf_prefix}${name}ar_gripper_finger1" />
+      <link name="${tf_prefix}${name}ar_gripper_finger2" />
+      <joint name="${tf_prefix}${name}ar_gripper_body_finger1" />
+      <passive_joint name="${tf_prefix}${name}ar_gripper_body_finger2" />
     </group>
     <!--LINKS - When a link is specified, the parent joint of that link (if it exists) is automatically included-->
@@ -20,21 +20,21 @@
     <!--SUBGROUPS - Groups can also be formed by referencing to already defined group names-->
     <!--GROUP STATES - Purpose - Define a named state for a particular group, in terms of joint values. This is useful to define states like 'folded arms'-->
-    <group_state name="close" group="${prefix}${name}ar_gripper">
-      <joint name="${prefix}${name}ar_gripper_body_finger1" value="0" />
-      <joint name="${prefix}${name}ar_gripper_body_finger2" value="0" />
+    <group_state name="close" group="${tf_prefix}${name}ar_gripper">
+      <joint name="${tf_prefix}${name}ar_gripper_body_finger1" value="0" />
+      <joint name="${tf_prefix}${name}ar_gripper_body_finger2" value="0" />
     </group_state>
-    <group_state name="open" group="${prefix}${name}ar_gripper">
-      <joint name="${prefix}${name}ar_gripper_body_finger1" value="0.05" />
-      <joint name="${prefix}${name}ar_gripper_body_finger2" value="0.05" />
+    <group_state name="open" group="${tf_prefix}${name}ar_gripper">
+      <joint name="${tf_prefix}${name}ar_gripper_body_finger1" value="0.05" />
+      <joint name="${tf_prefix}${name}ar_gripper_body_finger2" value="0.05" />
     </group_state>
     <!--END EFFECTOR - Purpose - Represent information about an end effector.-->
     <!--VIRTUAL JOINT - Purpose - this element defines a virtual joint between a robot link and an external frame of reference (considered fixed with respect to the robot)-->
     <!--DISABLE COLLISIONS - By default it is assumed that any link of the robot could potentially come into collision with any other link in the robot. This tag disables collision checking between a specified pair of links. -->
-    <disable_collisions link1="${prefix}${name}ar_gripper_adapter" link2="${prefix}${name}ar_gripper_body" reason="Adjacent" />
-    <disable_collisions link1="${prefix}${name}ar_gripper_adapter" link2="${prefix}${name}ar_gripper_finger1" reason="Never" />
-    <disable_collisions link1="${prefix}${name}ar_gripper_adapter" link2="${prefix}${name}ar_gripper_finger2" reason="Never" />
-    <disable_collisions link1="${prefix}${name}ar_gripper_body" link2="${prefix}${name}ar_gripper_finger1" reason="Adjacent" />
-    <disable_collisions link1="${prefix}${name}ar_gripper_body" link2="${prefix}${name}ar_gripper_finger2" reason="Adjacent" />
-    <disable_collisions link1="${prefix}${name}ar_gripper_finger1" link2="${prefix}${name}ar_gripper_finger2" reason="Adjacent" />
+    <disable_collisions link1="${tf_prefix}${name}ar_gripper_adapter" link2="${tf_prefix}${name}ar_gripper_body" reason="Adjacent" />
+    <disable_collisions link1="${tf_prefix}${name}ar_gripper_adapter" link2="${tf_prefix}${name}ar_gripper_finger1" reason="Never" />
+    <disable_collisions link1="${tf_prefix}${name}ar_gripper_adapter" link2="${tf_prefix}${name}ar_gripper_finger2" reason="Never" />
+    <disable_collisions link1="${tf_prefix}${name}ar_gripper_body" link2="${tf_prefix}${name}ar_gripper_finger1" reason="Adjacent" />
+    <disable_collisions link1="${tf_prefix}${name}ar_gripper_body" link2="${tf_prefix}${name}ar_gripper_finger2" reason="Adjacent" />
+    <disable_collisions link1="${tf_prefix}${name}ar_gripper_finger1" link2="${tf_prefix}${name}ar_gripper_finger2" reason="Adjacent" />
   </xacro:macro>
 </robot>

File: ar_gripper/urdf/ar_gripper_macro.xacro (robot description, xacro)
@@ -2,10 +2,10 @@
 <robot name="ar_gripper"
   xmlns:xacro="http://ros.org/wiki/xacro">
-  <xacro:macro name="ar_gripper_macro" params="prefix">
-    <material name="${prefix}Black">
+  <xacro:macro name="ar_gripper" params="tf_prefix">
+    <material name="${tf_prefix}Black">
       <color rgba="0.1 0.1 0.1 0.99"/>
     </material>
     <!-- link list -->
-    <link name="${prefix}ar_gripper_adapter">
+    <link name="${tf_prefix}ar_gripper_adapter">
       <visual>
         <geometry>
@@ -13,5 +13,5 @@
         </geometry>
         <origin rpy="0.0 0.0 0.0" xyz="0 0 0"/>
-        <material name="${prefix}Black">
+        <material name="${tf_prefix}Black">
         </material>
       </visual>
@@ -28,5 +28,5 @@
       </inertial>
     </link>
-    <link name="${prefix}ar_gripper_body">
+    <link name="${tf_prefix}ar_gripper_body">
       <visual>
         <geometry>
@@ -34,5 +34,5 @@
         </geometry>
         <origin rpy="0.0 0.0 0.0" xyz="0 0 0"/>
-        <material name="${prefix}Black">
+        <material name="${tf_prefix}Black">
         </material>
       </visual>
@@ -49,5 +49,5 @@
       </inertial>
     </link>
-    <link name="${prefix}ar_gripper_finger1">
+    <link name="${tf_prefix}ar_gripper_finger1">
       <visual>
         <geometry>
@@ -55,5 +55,5 @@
         </geometry>
         <origin rpy="0 0 0" xyz="0 0 0"/>
-        <material name="${prefix}Black">
+        <material name="${tf_prefix}Black">
         </material>
       </visual>
@@ -70,5 +70,5 @@
       </inertial>
     </link>
-    <link name="${prefix}ar_gripper_finger2">
+    <link name="${tf_prefix}ar_gripper_finger2">
       <visual>
         <geometry>
@@ -76,5 +76,5 @@
         </geometry>
         <origin rpy="0 0 0" xyz="0 0 0"/>
-        <material name="${prefix}Black">
+        <material name="${tf_prefix}Black">
         </material>
       </visual>
@@ -92,23 +92,23 @@
     </link>
     <!-- joint list -->
-    <joint name="${prefix}adapter_ar_gripper_body" type="fixed">
-      <parent link="${prefix}ar_gripper_adapter"/>
-      <child link="${prefix}ar_gripper_body"/>
+    <joint name="${tf_prefix}adapter_ar_gripper_body" type="fixed">
+      <parent link="${tf_prefix}ar_gripper_adapter"/>
+      <child link="${tf_prefix}ar_gripper_body"/>
       <axis xyz="0 0 0"/>
       <origin rpy="0 0 0" xyz="0 0 0.006"/>
     </joint>
-    <joint name="${prefix}ar_gripper_body_finger1" type="prismatic">
+    <joint name="${tf_prefix}ar_gripper_body_finger1" type="prismatic">
       <limit effort="1000.0" lower="0.0" upper="0.05" velocity="0.0031"/>
-      <parent link="${prefix}ar_gripper_body"/>
-      <child link="${prefix}ar_gripper_finger1"/>
+      <parent link="${tf_prefix}ar_gripper_body"/>
+      <child link="${tf_prefix}ar_gripper_finger1"/>
       <axis xyz="-1 0 0"/>
       <origin rpy="0 0 0" xyz="0.0 0 0.0756"/>
     </joint>
-    <joint name="${prefix}ar_gripper_body_finger2" type="prismatic">
+    <joint name="${tf_prefix}ar_gripper_body_finger2" type="prismatic">
       <limit effort="1000.0" lower="0.0" upper="0.05" velocity="0.0031"/>
-      <parent link="${prefix}ar_gripper_body"/>
-      <child link="${prefix}ar_gripper_finger2"/>
+      <parent link="${tf_prefix}ar_gripper_body"/>
+      <child link="${tf_prefix}ar_gripper_finger2"/>
       <axis xyz="-1 0 0"/>
-      <mimic joint="${prefix}ar_gripper_body_finger1" multiplier="1.0" offset="0.0" />
+      <mimic joint="${tf_prefix}ar_gripper_body_finger1" multiplier="1.0" offset="0.0" />
       <origin rpy="0 0 ${pi}" xyz="0.0 0 0.0756"/>
     </joint>

File: ar_gripper/urdf/ar_gripper_standalone.xacro (robot description, xacro)
@@ -2,5 +2,5 @@
 <robot name="za" xmlns:xacro="http://ros.org/wiki/xacro">
   <xacro:include filename="$(find ar_gripper)/urdf/ar_gripper_macro.xacro"/>
-  <xacro:ar_gripper_macro prefix="main_"/>
+  <xacro:ar_gripper tf_prefix="main_"/>
   <material name="main_Red">
     <color rgba="0.7 0.0 0.0 0.99"/>
