Commit message: Update meshes to match Fusion360 model. Refactor urdf to have swappable adapters. Add ur_adapter mesh.

File: ar_gripper/urdf/ar_gripper_macro.xacro (robot description, xacro)
@@ -2,5 +2,5 @@
 <robot name="ar_gripper"
   xmlns:xacro="http://ros.org/wiki/xacro">
-  <xacro:macro name="ar_gripper" params="tf_prefix sim:=false">
+  <xacro:macro name="ar_gripper" params="tf_prefix parent_link sim:=false">
     <!-- Workaround for https://github.com/ros-controls/gz_ros2_control/issues/165 -->
     <xacro:property name="FINGER_LOWER_LIMIT" value="0.0" />
@@ -8,29 +8,8 @@
     <xacro:property name="FINGER_ADJUSTED_LOWER_LIMIT" value="${FINGER_LOWER_LIMIT - 0.01}" />
     <xacro:property name="FINGER_ADJUSTED_UPPER_LIMIT" value="${FINGER_UPPER_LIMIT + 0.01}" />
+    <xacro:property name="FINGER_BODY_GAP" value="0.0005" />
     <material name="${tf_prefix}Black">
       <color rgba="0.1 0.1 0.1 0.99"/>
     </material>
-    <!-- link list -->
-    <link name="${tf_prefix}ar_gripper_adapter">
-      <visual>
-        <geometry>
-          <mesh filename="package://ar_gripper/meshes/adapter.stl"/>
-        </geometry>
-        <origin rpy="0.0 0.0 0.0" xyz="0 0 0"/>
-        <material name="${tf_prefix}Black">
-        </material>
-      </visual>
-      <collision>
-        <geometry>
-          <mesh filename="package://ar_gripper/meshes/adapter.stl"/>
-        </geometry>
-        <origin rpy="0.0 0.0 0.0" xyz="0 0 0"/>
-      </collision>
-      <inertial>
-        <mass value="0.040" />
-        <!-- These numbers are not correct -->
-        <inertia ixx="0.001" ixy="0.0" ixz="0.0" iyy="0.001" iyz="0.0" izz="0.001"/>
-      </inertial>
-    </link>
     <link name="${tf_prefix}ar_gripper_body">
       <visual>
@@ -54,4 +33,10 @@
       </inertial>
     </link>
+    <joint name="${tf_prefix}ar_gripper_parent_body" type="fixed">
+      <parent link="${parent_link}"/>
+      <child link="${tf_prefix}ar_gripper_body"/>
+      <axis xyz="0 0 0"/>
+      <origin rpy="0 0 0" xyz="0 0 0"/>
+    </joint>
     <link name="${tf_prefix}ar_gripper_finger1">
       <visual>
@@ -75,4 +60,12 @@
       </inertial>
     </link>
+    <joint name="${tf_prefix}ar_gripper_body_finger1" type="prismatic">
+      <limit effort="1000.0" lower="${FINGER_ADJUSTED_LOWER_LIMIT}" upper="${FINGER_ADJUSTED_UPPER_LIMIT}" velocity="0.0031"/>
+      <parent link="${tf_prefix}ar_gripper_body"/>
+      <child link="${tf_prefix}ar_gripper_finger1"/>
+      <axis xyz="-1 0 0"/>
+      <origin rpy="0 0 0" xyz="0.0 0 ${0.0756 + FINGER_BODY_GAP}"/>
+      <dynamics damping="0.3" />
+    </joint>
     <link name="${tf_prefix}ar_gripper_finger2">
       <visual>
@@ -96,19 +89,4 @@
       </inertial>
     </link>
-    <!-- joint list -->
-    <joint name="${tf_prefix}adapter_ar_gripper_body" type="fixed">
-      <parent link="${tf_prefix}ar_gripper_adapter"/>
-      <child link="${tf_prefix}ar_gripper_body"/>
-      <axis xyz="0 0 0"/>
-      <origin rpy="0 0 0" xyz="0 0 0.006"/>
-    </joint>
-    <joint name="${tf_prefix}ar_gripper_body_finger1" type="prismatic">
-      <limit effort="1000.0" lower="${FINGER_ADJUSTED_LOWER_LIMIT}" upper="${FINGER_ADJUSTED_UPPER_LIMIT}" velocity="0.0031"/>
-      <parent link="${tf_prefix}ar_gripper_body"/>
-      <child link="${tf_prefix}ar_gripper_finger1"/>
-      <axis xyz="-1 0 0"/>
-      <origin rpy="0 0 0" xyz="0.0 0 0.0756"/>
-      <dynamics damping="0.3" />
-    </joint>
     <joint name="${tf_prefix}ar_gripper_body_finger2" type="prismatic">
       <limit effort="1000.0" lower="${FINGER_ADJUSTED_LOWER_LIMIT}" upper="${FINGER_ADJUSTED_UPPER_LIMIT}" velocity="0.0031"/>
@@ -117,5 +95,5 @@
       <axis xyz="-1 0 0"/>
       <mimic joint="${tf_prefix}ar_gripper_body_finger1" multiplier="1.0" offset="0.0" />
-      <origin rpy="0 0 ${pi}" xyz="0.0 0 0.0756"/>
+      <origin rpy="0 0 ${pi}" xyz="0.0 0 ${0.0756 + FINGER_BODY_GAP}"/>
       <dynamics damping="0.3" />
     </joint>

File: ar_gripper/urdf/ar_gripper_standalone.xacro (robot description, xacro)
@@ -1,7 +1,9 @@
 <?xml version="1.0" ?>
-<robot name="za" xmlns:xacro="http://ros.org/wiki/xacro">
+<robot name="ar_gripper"
+  xmlns:xacro="http://ros.org/wiki/xacro">
   <xacro:include filename="$(find ar_gripper)/urdf/ar_gripper_macro.xacro"/>
-  <xacro:ar_gripper tf_prefix="main_"/>
-  <material name="main_Red">
+  <xacro:include filename="$(find ar_gripper)/urdf/ar_gripper_adapter_macro.xacro"/>
+  <xacro:property name="tf_prefix" value="main_" />
+  <material name="${tf_prefix}Red">
     <color rgba="0.7 0.0 0.0 0.99"/>
   </material>
@@ -13,5 +15,5 @@
       </geometry>
       <origin rpy="0 0 0" xyz="0 0 0.05"/>
-      <material name="main_Red"/>
+      <material name="${tf_prefix}Red"/>
     </visual>
   </link>
@@ -20,8 +22,12 @@
     <child link="base_link"/>
   </joint>
-  <joint name="base-adapter" type="fixed">
+  <link name="gripper_attachment" />
+  <joint name="base-gripper_attachment" type="fixed">
     <parent link="base_link"/>
-    <child link="main_ar_gripper_adapter"/>
+    <child link="gripper_attachment"/>
     <origin rpy="0 0 0" xyz="0 0 0.1"/>
   </joint>
+  <xacro:ar_gripper_adapter tf_prefix="${tf_prefix}" parent_link="gripper_attachment"/>
+  <!-- Inside whichever adapter is being used -->
+  <xacro:ar_gripper tf_prefix="${tf_prefix}" parent_link="${tf_prefix}ar_gripper_adapter_attachment"/>
 </robot>

File: ar_gripper/urdf/ar_gripper_standalone_sim.urdf.xacro (robot description, xacro)
@@ -3,6 +3,7 @@
   xmlns:xacro="http://ros.org/wiki/xacro">
   <xacro:include filename="$(find ar_gripper)/urdf/ar_gripper_macro.xacro"/>
-  <xacro:ar_gripper tf_prefix="primary_"/>
-  <material name="primary_Red">
+  <xacro:include filename="$(find ar_gripper)/urdf/ar_gripper_adapter_macro.xacro"/>
+  <xacro:property name="tf_prefix" value="primary_" />
+  <material name="${tf_prefix}Red">
     <color rgba="0.7 0.0 0.0 0.99"/>
   </material>
@@ -14,5 +15,5 @@
       </geometry>
       <origin rpy="0 0 0" xyz="0 0 0.05"/>
-      <material name="primary_Red"/>
+      <material name="${tf_prefix}Red"/>
     </visual>
   </link>
@@ -21,9 +22,13 @@
     <child link="base_link"/>
   </joint>
-  <joint name="base-adapter" type="fixed">
+  <link name="gripper_attachment" />
+  <joint name="base-gripper_attachment" type="fixed">
     <parent link="base_link"/>
-    <child link="primary_ar_gripper_adapter"/>
+    <child link="gripper_attachment"/>
     <origin rpy="0 0 0" xyz="0 0 0.1"/>
   </joint>
+  <xacro:ar_gripper_adapter tf_prefix="${tf_prefix}" parent_link="gripper_attachment"/>
+  <!-- Inside whichever adapter is being used -->
+  <xacro:ar_gripper tf_prefix="${tf_prefix}" parent_link="${tf_prefix}ar_gripper_adapter_attachment"/>
   <xacro:include filename="$(find ar_gripper)/urdf/ar_gripper_gz.ros2_control.xacro" />
   <xacro:ar_gripper_ros2_control name="primary" tf_prefix="" />
