Commit message: Fix round 2: finger velocity limit, sim time, and the executor that starved reads
The finger joint's velocity limit was 0.0031 m/s, which capped a full 0.05 m
stroke at 16 s and made it impossible to complete inside the driver's 20 s move
timeout. Nothing derives 0.0031; 3945 ticks over the stroke is 51.9 mm of travel
per motor revolution, so it is 3.6 rpm, and the drive speed the driver actually
writes (2450 steps/s) is 0.031 m/s = 36 rpm. Raised to 0.031 as an explicitly
provisional value pending a measurement on the real gripper.

- xacro: finger1/finger2 velocity 0.0031 -> 0.031, with the derivation and the
  provisional caveat in the description itself
- isaac_servo: read that limit out of the description instead of holding a
  fourth copy of it in a Python constant
- isaac_servo: ramp integrates the interval it measures, so its speed does not
  depend on the sim-time timer achieving its nominal rate
- isaac_servo: seed goal and published target from the first measured sample;
  they defaulted to 0.0, which is the closed stop, so the bus commanded a full
  close at startup wherever the finger was
- ar_gripper: simulator traffic moves to its own node on its own
  SingleThreadedExecutor. A 120 Hz subscription on a MultiThreadedExecutor
  delivers 53 Hz for a whole core with gaps to 700 ms, against 118 Hz for 0.13
  of a core and a 9 ms worst gap; that, not system jitter, is what made blocking
  reads time out. Replaces the temporary bootstrap executor
- ar_gripper: driver clock -> sim time via the same module seam mock.py uses;
  message stamps come from the simulator's clock
- ar_gripper: action server gets its own callback group, so a long grasp no
  longer blocks status, diagnostics and the overload check
- gripper: the inrush wait yields instead of spinning on a bare continue
- launch: plumb isaac_skip_calibration; make its bypass honest about what
  homing would have set
- tests: whole-node tests that go red if the executor split, the bootstrap
  spin, the velocity clamp, the callback groups or the seeding are removed

Live acceptance on a running stage: open -> close -> open all reached_goal with
zero joint-state timeouts, ~5.0 sim s per full stroke, driver at 11% CPU.

File: ar_gripper/urdf/ar_gripper_macro.xacro (robot description, xacro)
@@ -16,4 +16,24 @@
     <xacro:property name="FINGER_UPPER_LIMIT" value="0.05" />
     <xacro:property name="FINGER_BODY_GAP" value="0.0005" />
+    <!-- Finger velocity limit: PROVISIONAL, 0.031 m/s, and it MUST be confirmed by
+         timing a full open/close on the real gripper.
+         It is written as a literal on both <limit> elements below rather than as a
+         xacro property because the Isaac servo backend reads this file as plain XML to
+         avoid keeping a fourth copy of the number; a ${...} expression there would not
+         parse. If this ever has to become a property, teach that reader to expand
+         xacro instead of just moving the value.
+         Where 0.031 comes from. The finger's 0.05 m stroke spans 3945 encoder ticks on
+         a 4096 tick/rev encoder, i.e. 51.9 mm of finger travel per motor revolution.
+         The driver commands the servo at 122500 steps/s (Gripper._init_servo); the
+         value that actually goes on the wire is 122500 // 50 = 2450 steps/s, which at
+         78900 ticks/m is 0.031 m/s = 36 rpm. An STS3215 free-runs around 45 rpm, so
+         36 rpm loaded is mechanically sane.
+         The previous value here was 0.0031 m/s, i.e. 3.6 rpm, exactly 10x smaller.
+         Nothing derives it: `git log -S0.0031` finds no commit that introduced it, it
+         predates the directory move, and every timeout in gripper.py (the 20 s move
+         timeout, the 20 s wait-for-stop, the 0.3 s inrush window) is sized for a move
+         of order one second, not the 16 s a full stroke takes at 3.6 rpm. A dropped
+         decimal explains both numbers. Under Isaac the old value was binding and hard:
+         a full 0.05 m stroke could not complete inside the driver's own timeout. -->
     <material name="${tf_prefix}Black">
       <color rgba="0.1 0.1 0.1 0.99"/>
@@ -69,5 +89,5 @@
     </link>
     <joint name="${tf_prefix}ar_gripper_body_finger1" type="prismatic">
-      <limit effort="1000.0" lower="${FINGER_LOWER_LIMIT}" upper="${FINGER_UPPER_LIMIT}" velocity="0.0031"/>
+      <limit effort="1000.0" lower="${FINGER_LOWER_LIMIT}" upper="${FINGER_UPPER_LIMIT}" velocity="0.031"/>
       <parent link="${tf_prefix}ar_gripper_body"/>
       <child link="${tf_prefix}ar_gripper_finger1"/>
@@ -98,5 +118,5 @@
     </link>
     <joint name="${tf_prefix}ar_gripper_body_finger2" type="prismatic">
-      <limit effort="1000.0" lower="${FINGER_LOWER_LIMIT}" upper="${FINGER_UPPER_LIMIT}" velocity="0.0031"/>
+      <limit effort="1000.0" lower="${FINGER_LOWER_LIMIT}" upper="${FINGER_UPPER_LIMIT}" velocity="0.031"/>
       <parent link="${tf_prefix}ar_gripper_body"/>
       <child link="${tf_prefix}ar_gripper_finger2"/>
