Commit message: Use the finger's real travel limits, not the padded ones
The 10 mm padding at each end was a workaround for gz_ros2_control#165. It was
applied unconditionally, so a Gazebo workaround shipped in the real robot's
description, and it removed the only hard stop a simulator has: a homing routine
that closes until it feels load then finds nothing to push against.

Whether that Gazebo bug still exists is unverified and noted as such. Driving the
gripper limit-to-limit repeatedly on gz_ros2_control 1.2.19 did not reproduce any
sticking, but that is one rig, not a clearance.

Co-Authored-By: Claude Opus 5 (1M context) <noreply@anthropic.com>

File: ar_gripper/urdf/ar_gripper_macro.xacro (robot description, xacro)
@@ -3,9 +3,16 @@
   xmlns:xacro="http://ros.org/wiki/xacro">
   <xacro:macro name="ar_gripper" params="tf_prefix sim:=false">
-    <!-- Workaround for https://github.com/ros-controls/gz_ros2_control/issues/165 -->
+    <!-- These are the mechanism's real travel limits. They were previously padded by
+         10 mm at each end to work around
+         https://github.com/ros-controls/gz_ros2_control/issues/165 (a joint commanded
+         to its limit could stick there). The padding was unconditional, so a Gazebo
+         workaround also shipped in the real robot's description, and it removed the
+         only hard stop a simulator has - a gripper homing routine that closes until it
+         feels load then has nothing to push against.
+         Whether that Gazebo bug still exists on current gz_ros2_control is UNVERIFIED;
+         the upstream issue is still open and marked wontfix. If it resurfaces, gate the
+         padding on the simulator rather than applying it everywhere. -->
     <xacro:property name="FINGER_LOWER_LIMIT" value="0.0" />
     <xacro:property name="FINGER_UPPER_LIMIT" value="0.05" />
-    <xacro:property name="FINGER_ADJUSTED_LOWER_LIMIT" value="${FINGER_LOWER_LIMIT - 0.01}" />
-    <xacro:property name="FINGER_ADJUSTED_UPPER_LIMIT" value="${FINGER_UPPER_LIMIT + 0.01}" />
     <xacro:property name="FINGER_BODY_GAP" value="0.0005" />
     <material name="${tf_prefix}Black">
@@ -62,5 +69,5 @@
     </link>
     <joint name="${tf_prefix}ar_gripper_body_finger1" type="prismatic">
-      <limit effort="1000.0" lower="${FINGER_ADJUSTED_LOWER_LIMIT}" upper="${FINGER_ADJUSTED_UPPER_LIMIT}" velocity="0.0031"/>
+      <limit effort="1000.0" lower="${FINGER_LOWER_LIMIT}" upper="${FINGER_UPPER_LIMIT}" velocity="0.0031"/>
       <parent link="${tf_prefix}ar_gripper_body"/>
       <child link="${tf_prefix}ar_gripper_finger1"/>
@@ -91,5 +98,5 @@
     </link>
     <joint name="${tf_prefix}ar_gripper_body_finger2" type="prismatic">
-      <limit effort="1000.0" lower="${FINGER_ADJUSTED_LOWER_LIMIT}" upper="${FINGER_ADJUSTED_UPPER_LIMIT}" velocity="0.0031"/>
+      <limit effort="1000.0" lower="${FINGER_LOWER_LIMIT}" upper="${FINGER_UPPER_LIMIT}" velocity="0.0031"/>
       <parent link="${tf_prefix}ar_gripper_body"/>
       <child link="${tf_prefix}ar_gripper_finger2"/>

Commit message: Isaac Sim servo backend (#4)
Adds an Isaac Sim backend to the driver alongside the existing mock and
hardware paths, so the gripper can be driven in simulation without
changing anything the real robot runs.

- `IsaacServo` subclasses the offline mock at the byte level and takes
position and effort from the simulator instead of the internal travel
model
- simulator traffic runs on its own node and executor: a
`MultiThreadedExecutor` delivered 53 of 120 Hz while burning a full
core, where a single-threaded one delivers 118 Hz at 0.13
- homing detects the stop by motion, and treats a joint pinned at its
limit as stopped whatever its velocity says, because the drive keeps
reporting the velocity it wants
- "stopped" is decided over a window rather than between two samples:
Isaac publishes positions quantised to 1e-4, so a settling finger
repeats readings while still ~1.8 mm out and every move ended there with
`reached_goal` false
- `LOAD_DEADBAND_N` is derived from measured force rather than a Feetech
datasheet: 2.0 N sat between the finger's own weight (0.3924 N of steady
bias) and the weakest real grasp (1.599 N), so closing on a 400 g body
reported exactly zero load
- driver durations run on the simulator clock, with a wall-clock
backstop so a stopped simulator cannot hang a move
- the finger travel and velocity limits are read from the shipped
description rather than restated in code
- `mock.FakeServo` gains a motor-current model, a position-correlated
obstruction, and the first coverage of the current-stall branch, which
had never executed anywhere
- the test suite runs on its own ROS domain, after it was found to be
commanding a live simulator
- `gripper.py`, `feetech.py` and the wire behaviour of `mock.py` are
unchanged, so the real robot's homing is bit-for-bit what it was

The forces above are measured against a pinned finger collider in the
integrating workspace, with a grip-force tool that ships alongside the
simulator stage there. Its actuator parity test passes whole against a
live stage, gripper leg and exit codes included.

---------

Co-authored-by: Claude Opus 5 (1M context) <noreply@anthropic.com>

File: ar_gripper/urdf/ar_gripper_macro.xacro (robot description, xacro)
@@ -16,4 +16,44 @@
     <xacro:property name="FINGER_UPPER_LIMIT" value="0.05" />
     <xacro:property name="FINGER_BODY_GAP" value="0.0005" />
+    <!-- Finger velocity limit: PROVISIONAL, 0.031 m/s, and it MUST be confirmed by
+         timing a full open/close on the real gripper.
+         HOW TO CONFIRM IT, now that there is tooling for it. Attempted on
+         2026-08-16 and not completed: the gripper's servo cable had failed, so
+         nothing on the bus answered. Left for a follow-up.
+             ros2 launch ar_gripper ar_gripper_control.launch.py \
+                 bus_trace_path:=/tmp/gripper.csv bus_trace_sample_hz:=100
+             # drive several strokes of different lengths, then Ctrl-C
+             ros2 run ar_gripper analyze_bus_trace.py /tmp/gripper.csv
+         A full 0.05 m stroke takes about 1.6 s if this number is right and
+         about 16 s if the pre-2026-08 value of 0.0031 was, so the two are not
+         subtle to tell apart. What settles it is the reported cruise velocity,
+         not the stroke time: a stroke time also contains both ramps, the
+         driver's 0.3 s inrush window and its wait-for-stop dwell.
+         Also worth capturing in the same run, since the rig is set up: the
+         servo's acceleration register (0x29, `FeetechSMSServo.acceleration`,
+         steps/s^2) read back and compared against the acceleration the trace
+         implies. Nothing has ever checked that the configured value is what
+         the mechanism does. Sample at 100 Hz for that, because the driver's
+         own reads are 10 Hz during a move, which is roughly one sample of
+         ramp. Take one unsampled run alongside it: sampling adds bus traffic,
+         and the point is to measure the move rather than the measurement.
+         It is written as a literal on both <limit> elements below rather than as a
+         xacro property because the Isaac servo backend reads this file as plain XML to
+         avoid keeping a fourth copy of the number; a ${...} expression there would not
+         parse. If this ever has to become a property, teach that reader to expand
+         xacro instead of just moving the value.
+         Where 0.031 comes from. The finger's 0.05 m stroke spans 3945 encoder ticks on
+         a 4096 tick/rev encoder, i.e. 51.9 mm of finger travel per motor revolution.
+         The driver commands the servo at 122500 steps/s (Gripper._init_servo); the
+         value that actually goes on the wire is 122500 // 50 = 2450 steps/s, which at
+         78900 ticks/m is 0.031 m/s = 36 rpm. An STS3215 free-runs around 45 rpm, so
+         36 rpm loaded is mechanically sane.
+         The previous value here was 0.0031 m/s, i.e. 3.6 rpm, exactly 10x smaller.
+         Nothing derives it: `git log -S0.0031` finds no commit that introduced it, it
+         predates the directory move, and every timeout in gripper.py (the 20 s move
+         timeout, the 20 s wait-for-stop, the 0.3 s inrush window) is sized for a move
+         of order one second, not the 16 s a full stroke takes at 3.6 rpm. A dropped
+         decimal explains both numbers. Under Isaac the old value was binding and hard:
+         a full 0.05 m stroke could not complete inside the driver's own timeout. -->
     <!-- Alpha 1.0. An alpha below 1 is not a shading hint: it makes the
          surface transmissive, and a renderer has to trace through it. Under
@@ -74,5 +114,5 @@
     </link>
     <joint name="${tf_prefix}ar_gripper_body_finger1" type="prismatic">
-      <limit effort="1000.0" lower="${FINGER_LOWER_LIMIT}" upper="${FINGER_UPPER_LIMIT}" velocity="0.0031"/>
+      <limit effort="1000.0" lower="${FINGER_LOWER_LIMIT}" upper="${FINGER_UPPER_LIMIT}" velocity="0.031"/>
       <parent link="${tf_prefix}ar_gripper_body"/>
       <child link="${tf_prefix}ar_gripper_finger1"/>
@@ -103,5 +143,5 @@
     </link>
     <joint name="${tf_prefix}ar_gripper_body_finger2" type="prismatic">
-      <limit effort="1000.0" lower="${FINGER_LOWER_LIMIT}" upper="${FINGER_UPPER_LIMIT}" velocity="0.0031"/>
+      <limit effort="1000.0" lower="${FINGER_LOWER_LIMIT}" upper="${FINGER_UPPER_LIMIT}" velocity="0.031"/>
       <parent link="${tf_prefix}ar_gripper_body"/>
       <child link="${tf_prefix}ar_gripper_finger2"/>
