Commit message: Undo xacro parent_link pattern for more mounting flexibility

File: ar_gripper/urdf/ar_gripper_adapter_macro.xacro (robot description, xacro)
@@ -2,5 +2,6 @@
 <robot name="ar_gripper_adapter"
   xmlns:xacro="http://www.ros.org/wiki/xacro">
-  <xacro:macro name="ar_gripper_adapter" params="tf_prefix parent_link adapter_height:=0.006 adapter_mesh:=package://ar_gripper/meshes/adapter.stl">
+  <xacro:macro name="ar_gripper_adapter" params="tf_prefix adapter_height:=0.006 adapter_mesh:=package://ar_gripper/meshes/adapter.stl">
+    <link name="${tf_prefix}ar_gripper_adapter_mount" />
     <link name="${tf_prefix}ar_gripper_adapter">
       <visual>
@@ -24,6 +25,6 @@
       </inertial>
     </link>
-    <joint name="${tf_prefix}ar_gripper_parent_adapter" type="fixed">
-      <parent link="${parent_link}"/>
+    <joint name="${tf_prefix}ar_gripper_adapter_mount_adapter" type="fixed">
+      <parent link="${tf_prefix}ar_gripper_adapter_mount"/>
       <child link="${tf_prefix}ar_gripper_adapter"/>
       <axis xyz="0 0 0"/>

File: ar_gripper/urdf/ar_gripper_macro.xacro (robot description, xacro)
@@ -2,5 +2,5 @@
 <robot name="ar_gripper"
   xmlns:xacro="http://ros.org/wiki/xacro">
-  <xacro:macro name="ar_gripper" params="tf_prefix parent_link sim:=false">
+  <xacro:macro name="ar_gripper" params="tf_prefix sim:=false">
     <!-- Workaround for https://github.com/ros-controls/gz_ros2_control/issues/165 -->
     <xacro:property name="FINGER_LOWER_LIMIT" value="0.0" />
@@ -12,4 +12,5 @@
       <color rgba="0.1 0.1 0.1 0.99"/>
     </material>
+    <link name="${tf_prefix}ar_gripper_mount" />
     <link name="${tf_prefix}ar_gripper_body">
       <visual>
@@ -33,6 +34,6 @@
       </inertial>
     </link>
-    <joint name="${tf_prefix}ar_gripper_parent_body" type="fixed">
-      <parent link="${parent_link}"/>
+    <joint name="${tf_prefix}ar_gripper_mount_body" type="fixed">
+      <parent link="${tf_prefix}ar_gripper_mount"/>
       <child link="${tf_prefix}ar_gripper_body"/>
       <axis xyz="0 0 0"/>

File: ar_gripper/urdf/ar_gripper_standalone.xacro (robot description, xacro)
@@ -28,6 +28,17 @@
     <origin rpy="0 0 0" xyz="0 0 0.1"/>
   </joint>
-  <xacro:ar_gripper_adapter tf_prefix="${tf_prefix}" parent_link="gripper_attachment"/>
-  <!-- Inside whichever adapter is being used -->
-  <xacro:ar_gripper tf_prefix="${tf_prefix}" parent_link="${tf_prefix}ar_gripper_adapter_attachment"/>
+  <xacro:ar_gripper_adapter tf_prefix="${tf_prefix}"/>
+  <joint name="base-ar_gripper_adapter_mount" type="fixed">
+    <parent link="gripper_attachment"/>
+    <child link="${tf_prefix}ar_gripper_adapter_mount"/>
+    <axis xyz="0 0 0"/>
+    <origin rpy="0 0 0" xyz="0 0 0"/>
+  </joint>
+  <xacro:ar_gripper tf_prefix="${tf_prefix}"/>
+  <joint name="adapter_attachment-ar_gripper_mount" type="fixed">
+    <parent link="${tf_prefix}ar_gripper_adapter_attachment"/>
+    <child link="${tf_prefix}ar_gripper_mount"/>
+    <axis xyz="0 0 0"/>
+    <origin rpy="0 0 0" xyz="0 0 0"/>
+  </joint>
 </robot>

File: ar_gripper/urdf/ar_gripper_standalone_sim.urdf.xacro (robot description, xacro)
@@ -28,7 +28,18 @@
     <origin rpy="0 0 0" xyz="0 0 0.1"/>
   </joint>
-  <xacro:ar_gripper_adapter tf_prefix="${tf_prefix}" parent_link="gripper_attachment"/>
-  <!-- Inside whichever adapter is being used -->
-  <xacro:ar_gripper tf_prefix="${tf_prefix}" parent_link="${tf_prefix}ar_gripper_adapter_attachment"/>
+  <xacro:ar_gripper_adapter tf_prefix="${tf_prefix}"/>
+  <joint name="base-ar_gripper_adapter_mount" type="fixed">
+    <parent link="gripper_attachment"/>
+    <child link="${tf_prefix}ar_gripper_adapter_mount"/>
+    <axis xyz="0 0 0"/>
+    <origin rpy="0 0 0" xyz="0 0 0"/>
+  </joint>
+  <xacro:ar_gripper tf_prefix="${tf_prefix}"/>
+  <joint name="adapter_attachment-ar_gripper_mount" type="fixed">
+    <parent link="${tf_prefix}ar_gripper_adapter_attachment"/>
+    <child link="${tf_prefix}ar_gripper_mount"/>
+    <axis xyz="0 0 0"/>
+    <origin rpy="0 0 0" xyz="0 0 0"/>
+  </joint>
   <xacro:include filename="$(find ar_gripper)/urdf/ar_gripper_gz.ros2_control.xacro" />
   <xacro:ar_gripper_ros2_control name="primary" tf_prefix="" />
